File: Schema KiCad/PortePoulailler.kicad_pcb (KiCad board)
At the start: 2 copper layers, 78.7 x 51.4 mm, 14 parts, among them J1 FdcBas, J2 FdcHaut, J3 ConnecteurLed/Photoresistance, J4 +12V, J5 Connecteur moteur

Commit message: Mise a jour et début de rédaction de la notice
Parts:
- added D1: 1N5407, Diode_THT:D_DO-201AD_P5.08mm_Vertical_AnodeUp, F.Cu at (92.1, 64.1)
- R4: value 470ohm -> 180ohm
- moved R3 15.2 mm to (149.9, 82.5), turned to 90 degrees
Connections:
- J3 pad 4: GND -> +5V
- J4 pad 1: +12V -> Net-(D1-Pad2)
- R3 pad 1: +5V -> PhotoResistance
- R3 pad 2: PhotoResistance -> GND
Routing:
- net +12V: track 47.8 -> 68.6 mm
- net FdcBas: track 62.9 -> 44.7 mm
- net Net-(D1-Pad2): track 0.00 -> 6.35 mm
- net GND: track 261.9 -> 256.5 mm
- net +5V: track 149.9 -> 145.3 mm
Other:
- board text added: "Potar"
- board text added: "USB"
- board text added: "Ver. 1.1"
- board text removed: "Ver. 1.0"
