File: Schema KiCad/PortePoulailler.sch (KiCad schematic (older format))
At the start: 14 parts, among them J1 FdcBas, J2 FdcHaut, J3 ConnecteurLed/Photoresistance, J4 +12V, J5 Connecteur moteur

Commit message: Mise a jour et début de rédaction de la notice
Parts:
- added D1: 1N5407, Diode_THT:D_DO-201AD_P5.08mm_Vertical_AnodeUp, symbol Diode:1N5407
Connections:
- net +12V: now also D1.1 (K); no longer J4.1 (Pin_1)
- net +5V: now also J3.4 (Pin_4); no longer R3.1
- net GND: now also R3.2; no longer J3.4 (Pin_4)
- net PhotoResistance: now also R3.1; no longer R3.2
- new net: D1.2 (A), J4.1 (Pin_1)
Other:
- moved on the sheet: R3
Changed lines of the file:
@@
 L power:+12V #PWR0108
 U 1 1 5C8412BB
-P 7800 1700
-F 0 "#PWR0108" H 7800 1550 50  0001 C CNN
-F 1 "+12V" V 7815 1828 50  0000 L CNN
-F 2 "" H 7800 1700 50  0001 C CNN
-F 3 "" H 7800 1700 50  0001 C CNN
-	1    7800 1700
+P 7500 1700
+F 0 "#PWR0108" H 7500 1550 50  0001 C CNN
+F 1 "+12V" V 7515 1828 50  0000 L CNN
+F 2 "" H 7500 1700 50  0001 C CNN
+F 3 "" H 7500 1700 50  0001 C CNN
+	1    7500 1700
 	0    -1   -1   0
 $EndComp
@@
 L Device:R R3
 U 1 1 5C856740
-P 2850 1300
-F 0 "R3" H 2650 1400 50  0000 L CNN
-F 1 "10K" H 2450 1300 50  0000 L CNN
-F 2 "Resistor_THT:R_Axial_DIN0414_L11.9mm_D4.5mm_P15.24mm_Horizontal" V 2780 1300 50  0001 C CNN
-F 3 "~" H 2850 1300 50  0001 C CNN
-	1    2850 1300
-	1    0    0    -1
+P 2950 1300
+F 0 "R3" V 2950 1250 50  0000 L CNN
+F 1 "10K" H 3050 1300 50  0000 L CNN
+F 2 "Resistor_THT:R_Axial_DIN0414_L11.9mm_D4.5mm_P15.24mm_Horizontal" V 2880 1300 50  0001 C CNN
+F 3 "~" H 2950 1300 50  0001 C CNN
+	1    2950 1300
+	-1   0    0    1
 $EndComp
 $Comp
 L power:+5V #PWR0113
 U 1 1 5C8567EF
-P 2850 1150
-F 0 "#PWR0113" H 2850 1000 50  0001 C CNN
-F 1 "+5V" H 2865 1323 50  0000 C CNN
-F 2 "" H 2850 1150 50  0001 C CNN
-F 3 "" H 2850 1150 50  0001 C CNN
-	1    2850 1150
-	1    0    0    -1
-$EndComp
-Text GLabel 2550 1450 0    50   Input ~ 0
+P 3150 1350
+F 0 "#PWR0113" H 3150 1200 50  0001 C CNN
+F 1 "+5V" H 3150 1500 50  0000 C CNN
+F 2 "" H 3150 1350 50  0001 C CNN
+F 3 "" H 3150 1350 50  0001 C CNN
+	1    3150 1350
+	1    0    0    -1
+$EndComp
+Text GLabel 2850 1450 0    50   Input ~ 0
 PhotoResistance
 Text GLabel 5500 3400 2    50   Input ~ 0
@@
 U 1 1 5C88D5CF
 P 3100 1650
-F 0 "R4" V 3200 1550 50  0000 C CNN
-F 1 "180ohm" V 3200 1800 50  0000 C CNN
+F 0 "R4" V 3100 1650 50  0000 C CNN
+F 1 "180ohm" V 3200 1650 50  0000 C CNN
 F 2 "Resistor_THT:R_Axial_DIN0414_L11.9mm_D4.5mm_P15.24mm_Horizontal" V 3030 1650 50  0001 C CNN
 F 3 "~" H 3100 1650 50  0001 C CNN
@@
 L power:GND #PWR0119
 U 1 1 5C8918D9
-P 3250 1350
-F 0 "#PWR0119" H 3250 1100 50  0001 C CNN
-F 1 "GND" V 3255 1222 50  0000 R CNN
-F 2 "" H 3250 1350 50  0001 C CNN
-F 3 "" H 3250 1350 50  0001 C CNN
-	1    3250 1350
-	0    1    1    0
-$EndComp
-Wire Wire Line
-	2850 1450 3250 1450
-Wire Wire Line
-	2550 1450 2850 1450
-Connection ~ 2850 1450
+P 2950 1150
+F 0 "#PWR0119" H 2950 900 50  0001 C CNN
+F 1 "GND" H 3050 1000 50  0000 R CNN
+F 2 "" H 2950 1150 50  0001 C CNN
+F 3 "" H 2950 1150 50  0001 C CNN
+	1    2950 1150
+	-1   0    0    1
+$EndComp
+Wire Wire Line
+	2850 1450 2950 1450
+Wire Wire Line
+	3150 1350 3250 1350
+Wire Wire Line
+	2950 1450 3250 1450
+Connection ~ 2950 1450
+$Comp
+L Diode:1N5407 D1
+U 1 1 5D6A7FA8
+P 7650 1700
+F 0 "D1" H 7650 1916 50  0000 C CNN
+F 1 "1N5407" H 7650 1825 50  0000 C CNN
+F 2 "Diode_THT:D_DO-201AD_P5.08mm_Vertical_AnodeUp" H 7650 1525 50  0001 C CNN
+F 3 "http://www.vishay.com/docs/88516/1n5400.pdf" H 7650 1700 50  0001 C CNN
+	1    7650 1700
+	1    0    0    -1
+$EndComp
 $EndSCHEMATC
